Commit message: completed robot... for now

File: src/ros2_ws/src/rotom_description/urdf/rotom.urdf.xacro (robot description, xacro)
@@ -51,5 +51,5 @@
   <link name="wrist_flick">
     <visual>
-      <origin xyz="0.0206 0 -0.01285" rpy="3.14159265359 0 0"/>
+      <origin xyz="0.0206 0 -0.01285" rpy="0 0 0"/>
       <material name="gray"/>
       <geometry>
@@ -61,8 +61,18 @@
   <link name="flick_claw">
     <visual>
-      <origin xyz="0 0 0" rpy="0 0 0"/>
+      <origin xyz="0 0.0405 0" rpy="0 0 0"/>
       <material name="blue"/>
       <geometry>
         <mesh filename="package://rotom_description/meshes/visual/flick2claw.stl"
+              scale="${mesh_scale} ${mesh_scale} ${mesh_scale}"/>
+      </geometry>
+    </visual>
+  </link>
+  <link name="ee">
+    <visual>
+      <origin xyz="0 0.003 0" rpy="0 0 0"/>
+      <material name="gray"/>
+      <geometry>
+        <mesh filename="package://rotom_description/meshes/visual/EE.stl"
               scale="${mesh_scale} ${mesh_scale} ${mesh_scale}"/>
       </geometry>
@@ -100,5 +110,11 @@
     <parent link="wrist_flick"/>
     <child link="flick_claw"/>
-    <origin xyz="0.0206 0 0" rpy="0 0 0"/>
+    <origin xyz="0.0206 -0.01825 0.02265" rpy="0 0 0"/>
+    <axis xyz="0 1 0"/>
+  </joint>
+  <joint name="flick_to_ee" type="continuous">
+    <parent link="flick_claw"/>
+    <child link="ee"/>
+    <origin xyz="0.0668 0.0365 0" rpy="0 0 0"/>
     <axis xyz="0 1 0"/>
   </joint>

Commit message: control note + moveit tuning

File: src/ros2_ws/src/rotom_description/urdf/rotom.urdf.xacro (robot description, xacro)
@@ -79,4 +79,13 @@
     </visual>
   </link>
+  <link name="tool0">
+    <visual>
+      <origin xyz="0 0 0" rpy="0 0 0"/>
+      <geometry>
+        <box size="0.01 0.01 0.01"/>
+      </geometry>
+      <material name="gray"/>
+    </visual>
+  </link>
   <joint name="world_to_base" type="fixed">
     <parent link="world"/>
@@ -125,3 +134,8 @@
     <limit lower="-1.57" upper="1.57" effort="5.0" velocity="3.0"/>
   </joint>
+  <joint name="tool0" type="fixed">
+    <parent link="ee"/>
+    <child link="tool0"/>
+    <origin xyz="0.055 -.01825 0" rpy="0 0 0"/>
+  </joint>
 </robot>

Commit message: control works!!

File: src/ros2_ws/src/rotom_description/urdf/rotom.urdf.xacro (robot description, xacro)
@@ -18,4 +18,11 @@
       </geometry>
     </visual>
+    <collision>
+      <origin xyz="0 0 0" rpy="0 0 0"/>
+      <geometry>
+        <mesh filename="package://rotom_description/meshes/visual/origin2base.stl"
+              scale="${mesh_scale} ${mesh_scale} ${mesh_scale}"/>
+      </geometry>
+    </collision>
   </link>
   <link name="base_shoulder">
@@ -28,4 +35,11 @@
       </geometry>
     </visual>
+    <collision>
+      <origin xyz="0.0166 0 -0.01285" rpy="0 0 0"/>
+      <geometry>
+        <mesh filename="package://rotom_description/meshes/visual/base2shoulder.stl"
+              scale="${mesh_scale} ${mesh_scale} ${mesh_scale}"/>
+      </geometry>
+    </collision>
   </link>
   <link name="shoulder_elbow">
@@ -38,4 +52,11 @@
       </geometry>
     </visual>
+    <collision>
+      <origin xyz="0 0.0405 0" rpy="0 0 0"/>
+      <geometry>
+        <mesh filename="package://rotom_description/meshes/visual/shoulder2elbow.stl"
+              scale="${mesh_scale} ${mesh_scale} ${mesh_scale}"/>
+      </geometry>
+    </collision>
   </link>
   <link name="elbow_wrist">
@@ -48,4 +69,11 @@
       </geometry>
     </visual>
+    <collision>
+      <origin xyz="0 -0.006 0" rpy="3.14159265359 0 0"/>
+      <geometry>
+        <mesh filename="package://rotom_description/meshes/visual/elbow2wrist.stl"
+              scale="${mesh_scale} ${mesh_scale} ${mesh_scale}"/>
+      </geometry>
+    </collision>
   </link>
   <link name="wrist_flick">
@@ -58,4 +86,11 @@
       </geometry>
     </visual>
+    <collision>
+      <origin xyz="0.0206 0 -0.01285" rpy="0 0 0"/>
+      <geometry>
+        <mesh filename="package://rotom_description/meshes/visual/wrist2flick.stl"
+              scale="${mesh_scale} ${mesh_scale} ${mesh_scale}"/>
+      </geometry>
+    </collision>
   </link>
   <link name="flick_claw">
@@ -68,4 +103,11 @@
       </geometry>
     </visual>
+    <collision>
+      <origin xyz="0 0.0405 0" rpy="0 0 0"/>
+      <geometry>
+        <mesh filename="package://rotom_description/meshes/visual/flick2claw.stl"
+              scale="${mesh_scale} ${mesh_scale} ${mesh_scale}"/>
+      </geometry>
+    </collision>
   </link>
   <link name="ee">
@@ -78,4 +120,11 @@
       </geometry>
     </visual>
+    <collision>
+      <origin xyz="0 0.003 0" rpy="0 0 0"/>
+      <geometry>
+        <mesh filename="package://rotom_description/meshes/visual/EE.stl"
+              scale="${mesh_scale} ${mesh_scale} ${mesh_scale}"/>
+      </geometry>
+    </collision>
   </link>
   <link name="tool0">
@@ -87,4 +136,10 @@
       <material name="gray"/>
     </visual>
+    <collision>
+      <origin xyz="0 0 0" rpy="0 0 0"/>
+      <geometry>
+        <box size="0.01 0.01 0.01"/>
+      </geometry>
+    </collision>
   </link>
   <joint name="world_to_base" type="fixed">
@@ -97,5 +152,5 @@
     <origin xyz="0 -0.03 0.04025" rpy="1.570796 -1.570796 0"/>
     <axis xyz="1 0 0"/>
-    <limit lower="-3.14159" upper="3.14159" effort="5.0" velocity="3.0"/>
+    <limit lower="-3.141593" upper="3.141593" effort="5.0" velocity="3.0"/>
   </joint>
   <joint name="shoulder_to_elbow" type="revolute">
@@ -104,5 +159,5 @@
     <origin xyz="0.0166 -0.01825 0.02265" rpy="0 0 0"/>
     <axis xyz="0 1 0"/>
-    <limit lower="-2.2" upper="2.2" effort="5.0" velocity="3.0"/>
+    <limit lower="-0.055237" upper="0.823949" effort="5.0" velocity="3.0"/>
   </joint>
   <joint name="elbow_to_wrist" type="revolute">
@@ -111,5 +166,5 @@
     <origin xyz="0.0868 0 0" rpy="0 0 0"/>
     <axis xyz="0 1 0"/>
-    <limit lower="-2.2" upper="2.2" effort="5.0" velocity="3.0"/>
+    <limit lower="-1.410073" upper="1.997731" effort="5.0" velocity="3.0"/>
   </joint>
   <joint name="wrist_to_flick" type="revolute">
@@ -118,5 +173,5 @@
     <origin xyz="0.06025 0.01825 -0.0285" rpy="0 0 0"/>
     <axis xyz="1 0 0"/>
-    <limit lower="-2.0" upper="2.0" effort="5.0" velocity="3.0"/>
+    <limit lower="-3.141593" upper="3.141593" effort="5.0" velocity="3.0"/>
   </joint>
   <joint name="flick_to_claw" type="revolute">
@@ -125,5 +180,5 @@
     <origin xyz="0.0206 -0.01825 0.02265" rpy="0 0 0"/>
     <axis xyz="0 1 0"/>
-    <limit lower="-1.57" upper="1.57" effort="5.0" velocity="3.0"/>
+    <limit lower="-0.306871" upper="1.647898" effort="5.0" velocity="3.0"/>
   </joint>
   <joint name="flick_to_ee" type="revolute">
@@ -132,5 +187,5 @@
     <origin xyz="0.0668 0.0365 0" rpy="0 0 0"/>
     <axis xyz="0 1 0"/>
-    <limit lower="-1.57" upper="1.57" effort="5.0" velocity="3.0"/>
+    <limit lower="-1.884188" upper="1.885723" effort="5.0" velocity="3.0"/>
   </joint>
   <joint name="tool0" type="fixed">

File: src/ros2_ws/src/rotom_moveit_config/config/rotom.urdf.xacro (robot description, xacro)
@@ -2,8 +2,11 @@
 <robot xmlns:xacro="http://www.ros.org/wiki/xacro" name="rotom">
     <xacro:arg name="initial_positions_file" default="initial_positions.yaml" />
+    <xacro:arg name="use_ros2_control" default="false" />
     <!-- Import rotom urdf file -->
     <xacro:include filename="$(find rotom_description)/urdf/rotom.urdf.xacro" />
-    <!-- Import control_xacro -->
-    <xacro:include filename="rotom.ros2_control.xacro" />
-    <xacro:rotom_ros2_control name="FakeSystem" initial_positions_file="$(arg initial_positions_file)"/>
+    <xacro:if value="$(arg use_ros2_control)">
+        <!-- Import control_xacro -->
+        <xacro:include filename="rotom.ros2_control.xacro" />
+        <xacro:rotom_ros2_control name="FakeSystem" initial_positions_file="$(arg initial_positions_file)"/>
+    </xacro:if>
 </robot>

Commit message: recalibrate

File: src/ros2_ws/src/rotom_description/urdf/rotom.urdf.xacro (robot description, xacro)
@@ -159,5 +159,5 @@
     <origin xyz="0.0166 -0.01825 0.02265" rpy="0 0 0"/>
     <axis xyz="0 1 0"/>
-    <limit lower="-0.055237" upper="0.823949" effort="5.0" velocity="3.0"/>
+    <limit lower="-0.446497" upper="0.322215" effort="5.0" velocity="3.0"/>
   </joint>
   <joint name="elbow_to_wrist" type="revolute">
@@ -166,5 +166,5 @@
     <origin xyz="0.0868 0 0" rpy="0 0 0"/>
     <axis xyz="0 1 0"/>
-    <limit lower="-1.410073" upper="1.997731" effort="5.0" velocity="3.0"/>
+    <limit lower="-1.410073" upper="2.192594" effort="5.0" velocity="3.0"/>
   </joint>
   <joint name="wrist_to_flick" type="revolute">
@@ -180,5 +180,5 @@
     <origin xyz="0.0206 -0.01825 0.02265" rpy="0 0 0"/>
     <axis xyz="0 1 0"/>
-    <limit lower="-0.306871" upper="1.647898" effort="5.0" velocity="3.0"/>
+    <limit lower="-0.348299" upper="1.480653" effort="5.0" velocity="3.0"/>
   </joint>
   <joint name="flick_to_ee" type="revolute">
@@ -187,5 +187,5 @@
     <origin xyz="0.0668 0.0365 0" rpy="0 0 0"/>
     <axis xyz="0 1 0"/>
-    <limit lower="-1.884188" upper="1.885723" effort="5.0" velocity="3.0"/>
+    <limit lower="-2.023815" upper="2.178785" effort="5.0" velocity="3.0"/>
   </joint>
   <joint name="tool0" type="fixed">

Commit message: first motor in. now setting up servo control. hopefully moveit works

File: src/ros2_ws/src/rotom_description/urdf/rotom.urdf.xacro (robot description, xacro)
@@ -2,6 +2,6 @@
 <robot name="rotom" xmlns:xacro="http://www.ros.org/wiki/xacro">
   <xacro:property name="mesh_scale" value="0.001"/>
-    <material name="black">
-        <color rgba="0.0 0.0 0.0 1.0"/>
+    <material name="gray">
+        <color rgba="0.5 0.5 0.5 1.0"/>
     </material>
     <material name="yellow">
@@ -21,5 +21,5 @@
     <visual>
       <origin xyz="0 0 0" rpy="0 0 0"/>
-      <material name="black"/>
+      <material name="gray"/>
       <geometry>
         <mesh filename="package://rotom_description/meshes/visual/ground.stl"
@@ -30,5 +30,5 @@
       <origin xyz="0 0 0" rpy="0 0 0"/>
       <geometry>
-        <mesh filename="package://rotom_description/meshes/visual/origin2base.stl"
+        <mesh filename="package://rotom_description/meshes/visual/ground.stl"
               scale="${mesh_scale} ${mesh_scale} ${mesh_scale}"/>
       </geometry>
@@ -38,5 +38,6 @@
     <visual>
     <!---1.570796-->
-      <origin xyz="0.0166 0 -0.01285" rpy="0 0 0"/>
+      <origin xyz="0.05 0.012 -0.023" rpy="0 0 0"/>
+      <material name="red"/>
       <geometry>
         <mesh filename="package://rotom_description/meshes/visual/link1.stl"
@@ -45,5 +46,5 @@
     </visual>
     <collision>
-      <origin xyz="0.0166 0 -0.01285" rpy="0 0 0"/>
+      <origin xyz="0.05 0.012 -0.023" rpy="0 0 0"/>
       <geometry>
         <mesh filename="package://rotom_description/meshes/visual/link1.stl"
@@ -59,6 +60,6 @@
     <parent link="ground"/>
     <child link="link1"/>
-    <origin xyz="0 -0.03 0.04025" rpy="1.570796 -1.570796 0"/>
-    <axis xyz="1 0 0"/>
+    <origin xyz="0 0.02 0.0292" rpy="0 0 1.570796"/>
+    <axis xyz="0 0 1"/>
     <limit lower="-3.141593" upper="3.141593" effort="5.0" velocity="3.0"/>
   </joint>

Commit message: moveit set up with new robot

File: src/ros2_ws/src/rotom_description/urdf/rotom.urdf.xacro (robot description, xacro)
@@ -37,5 +37,4 @@
   <link name="link1">
     <visual>
-    <!---1.570796-->
       <origin xyz="0.05 0.012 -0.023" rpy="0 0 0"/>
       <material name="red"/>
@@ -53,4 +52,36 @@
     </collision>
   </link>
+  <link name="link2">
+    <visual>
+      <origin xyz="0.0 0.02 -0.011" rpy="0 0 0"/>
+      <material name="green"/>
+      <geometry>
+        <mesh filename="package://rotom_description/meshes/visual/link2.stl"
+              scale="${mesh_scale} ${mesh_scale} ${mesh_scale}"/>
+      </geometry>
+    </visual>
+    <collision>
+      <origin xyz="0.0 0.02 -0.011" rpy="0 0 0"/>
+      <geometry>
+        <mesh filename="package://rotom_description/meshes/visual/link2.stl"
+              scale="${mesh_scale} ${mesh_scale} ${mesh_scale}"/>
+      </geometry>
+    </collision>
+  </link>
+  <link name="tool0">
+    <visual>
+      <origin xyz="0 0 0" rpy="0 0 0"/>
+      <geometry>
+        <box size="0.01 0.01 0.01"/>
+      </geometry>
+      <material name="gray"/>
+    </visual>
+    <collision>
+      <origin xyz="0 0 0" rpy="0 0 0"/>
+      <geometry>
+        <box size="0.01 0.01 0.01"/>
+      </geometry>
+    </collision>
+  </link>
   <joint name="ground" type="fixed">
     <parent link="world"/>
@@ -62,5 +93,17 @@
     <origin xyz="0 0.02 0.0292" rpy="0 0 1.570796"/>
     <axis xyz="0 0 1"/>
-    <limit lower="-3.141593" upper="3.141593" effort="5.0" velocity="3.0"/>
+    <limit lower="-1.787524" upper="1.787524" effort="5.0" velocity="3.0"/>
+  </joint>
+  <joint name="A" type="revolute">
+    <parent link="link1"/>
+    <child link="link2"/>
+    <origin xyz="0.0344 0 0.0615" rpy="0 0 1.570796"/>
+    <axis xyz="-1 0 0"/>
+    <limit lower="-3.141593" upper="0.405070" effort="5.0" velocity="3.0"/>
+  </joint>
+  <joint name="B" type="fixed">
+    <parent link="link2"/>
+    <child link="tool0"/>
+    <origin xyz="0 0.0996 0.029" rpy="0 0 0"/>
   </joint>
 </robot>

Commit message: aruco following works

File: src/ros2_ws/src/rotom_description/urdf/rotom.urdf.xacro (robot description, xacro)
@@ -54,5 +54,5 @@
   <link name="link2">
     <visual>
-      <origin xyz="0.0 0.02 -0.011" rpy="0 0 0"/>
+      <origin xyz="0.0 0.02 -0.012" rpy="0 0 0"/>
       <material name="green"/>
       <geometry>
@@ -62,7 +62,41 @@
     </visual>
     <collision>
-      <origin xyz="0.0 0.02 -0.011" rpy="0 0 0"/>
+      <origin xyz="0.0 0.02 -0.012" rpy="0 0 0"/>
       <geometry>
         <mesh filename="package://rotom_description/meshes/visual/link2.stl"
+              scale="${mesh_scale} ${mesh_scale} ${mesh_scale}"/>
+      </geometry>
+    </collision>
+  </link>
+    <link name="link3">
+    <visual>
+      <origin xyz="0.0 0.02 -0.012" rpy="0 0 0"/>
+      <material name="blue"/>
+      <geometry>
+        <mesh filename="package://rotom_description/meshes/visual/link3.stl"
+              scale="${mesh_scale} ${mesh_scale} ${mesh_scale}"/>
+      </geometry>
+    </visual>
+    <collision>
+      <origin xyz="0.0 0.02 -0.012" rpy="0 0 0"/>
+      <geometry>
+        <mesh filename="package://rotom_description/meshes/visual/link3.stl"
+              scale="${mesh_scale} ${mesh_scale} ${mesh_scale}"/>
+      </geometry>
+    </collision>
+  </link>
+  <link name="link4">
+    <visual>
+      <origin xyz="0.0 0.02 -0.012" rpy="0 0 0"/>
+      <material name="yellow"/>
+      <geometry>
+        <mesh filename="package://rotom_description/meshes/visual/link4.stl"
+              scale="${mesh_scale} ${mesh_scale} ${mesh_scale}"/>
+      </geometry>
+    </visual>
+    <collision>
+      <origin xyz="0.0 0.02 -0.012" rpy="0 0 0"/>
+      <geometry>
+        <mesh filename="package://rotom_description/meshes/visual/link4.stl"
               scale="${mesh_scale} ${mesh_scale} ${mesh_scale}"/>
       </geometry>
@@ -102,8 +136,22 @@
     <limit lower="-3.141593" upper="0.405070" effort="5.0" velocity="3.0"/>
   </joint>
-  <joint name="B" type="fixed">
+  <joint name="B" type="revolute">
     <parent link="link2"/>
+    <child link="link3"/>
+    <origin xyz="0 0.0996 0.029" rpy="3.141593 0 0"/>
+    <axis xyz="-1 0 0"/>
+    <limit lower="-0.0421948" upper="3.141593" effort="5.0" velocity="3.0"/>
+  </joint>
+  <joint name="C" type="revolute">
+    <parent link="link3"/>
+    <child link="link4"/>
+    <origin xyz="0 0.1215 0.0" rpy="-1.570796 0 0"/>
+    <axis xyz="-1 0 0"/>
+    <limit lower="-3.141593" upper="0.377451" effort="5.0" velocity="3.0"/>
+  </joint>
+  <joint name="tool0_fixed" type="fixed">
+    <parent link="link4"/>
     <child link="tool0"/>
-    <origin xyz="0 0.0996 0.029" rpy="0 0 0"/>
+    <origin xyz="0 0.064 0.0" rpy="-1.570796 0 -1.570796"/>
   </joint>
 </robot>

File: src/ros2_ws/src/rotom_moveit_config/config/rotom.ros2_control.xacro (robot description, xacro)
@@ -22,4 +22,18 @@
                 <state_interface name="velocity"/>
             </joint>
+            <joint name="B">
+                <command_interface name="position"/>
+                <state_interface name="position">
+                  <param name="initial_value">${initial_positions['B']}</param>
+                </state_interface>
+                <state_interface name="velocity"/>
+            </joint>
+            <joint name="C">
+                <command_interface name="position"/>
+                <state_interface name="position">
+                  <param name="initial_value">${initial_positions['C']}</param>
+                </state_interface>
+                <state_interface name="velocity"/>
+            </joint>
         </ros2_control>
     </xacro:macro>
